Commit message: updated

File: zed_wrapper/urdf/include/materials.urdf.xacro (robot description, xacro)
@@ -16,15 +16,6 @@
 -->
 <robot>
-    <material name="zed_mat">
-        <color rgba="0.8 0.8 0.8 0.8"/>
-    </material>
-    <material name="zedm_mat">
-        <color rgba="0 0 0 0.9"/>
-    </material>
     <material name="zed2_mat">
         <color rgba="0.25 0.25 0.25 0.99"/>
     </material>
-    <material name="zed2i_mat">
-        <color rgba="0.25 0.25 0.25 0.99"/>
-    </material>
 </robot>

File: zed_wrapper/urdf/zed_descr.urdf.xacro (robot description, xacro)
@@ -18,5 +18,4 @@
   <xacro:arg name="camera_name"   default="zed" />
   <xacro:arg name="camera_model"  default="zed" />
-  <xacro:arg name="base_frame"    default="base_link" />
   <xacro:arg name="cam_pos_x"     default="0.0" />
   <xacro:arg name="cam_pos_y"     default="0.0" />

File: zed_wrapper/urdf/zed_macro.urdf.xacro (robot description, xacro)
@@ -26,18 +26,4 @@
   -->
   <xacro:macro name="zed_camera" params="name=zed model=zed parent *origin">
-    <xacro:if value="${model == 'zed'}">
-      <xacro:property name="baseline" value="0.12" />
-      <xacro:property name="height" value="0.03" />
-      <xacro:property name="bottom_slope" value="0.05" />
-      <xacro:property name="screw_offset_x" value="0.0" />
-      <xacro:property name="optical_offset_x" value="-0.01" />
-    </xacro:if>
-    <xacro:if value="${model == 'zedm'}">
-      <xacro:property name="baseline" value="0.06" />
-      <xacro:property name="height" value="0.0265" />
-      <xacro:property name="bottom_slope" value="0.0" />
-      <xacro:property name="screw_offset_x" value="0.0" />
-      <xacro:property name="optical_offset_x" value="0.0" />
-    </xacro:if>
     <xacro:if value="${model == 'zed2'}">
       <xacro:property name="baseline" value="0.12" />
@@ -45,11 +31,4 @@
       <xacro:property name="bottom_slope" value="0.05" />
       <xacro:property name="screw_offset_x" value="0.0" />
-      <xacro:property name="optical_offset_x" value="-0.01" />
-    </xacro:if>
-    <xacro:if value="${model == 'zed2i'}">
-      <xacro:property name="baseline" value="0.12" />
-      <xacro:property name="height" value="0.03" />
-      <xacro:property name="bottom_slope" value="0.0" />
-      <xacro:property name="screw_offset_x" value="-0.01" />
       <xacro:property name="optical_offset_x" value="-0.01" />
     </xacro:if>
